Commit message: Complete Assignemnt 5

File: body.urdf (robot description, URDF)
Before this commit: robot robot, 9 links, 8 joints
Links:
- removed link BackLeg
- removed link BackLowerLeg
- removed link FrontLeg
- removed link FrontLowerLeg
- removed link LeftLeg
- removed link LeftLowerLeg
- removed link RightLeg
- removed link RightLowerLeg
- added link LeftCalf, mass 1; collision box size=0.2 0.2 0.6; visual box size=0.2 0.2 0.6
- added link LeftFoot, mass 1; collision box size=0.5 0.5 0.05; visual box size=0.5 0.5 0.05
- added link LeftThigh, mass 1; collision box size=0.2 0.2 0.6; visual box size=0.2 0.2 0.6
- added link RightCalf, mass 1; collision box size=0.2 0.2 0.6; visual box size=0.2 0.2 0.6
- added link RightFoot, mass 1; collision box size=0.5 0.5 0.05; visual box size=0.5 0.5 0.05
- added link RightThigh, mass 1; collision box size=0.2 0.2 0.6; visual box size=0.2 0.2 0.6
- link Torso: geometry collision box size=0.6 0.4 0.3; visual box size=0.6 0.4 0.3
Joints:
- removed joint BackLeg_BackLowerLeg
- removed joint FrontLeg_FrontLowerLeg
- removed joint LeftLeg_LeftLowerLeg
- removed joint RightLeg_RightLowerLeg
- removed joint Torso_BackLeg
- removed joint Torso_FrontLeg
- removed joint Torso_LeftLeg
- removed joint Torso_RightLeg
- added joint LeftCalf_LeftFoot: type revolute, parent LeftCalf, child LeftFoot, origin xyz=0 0 -0.5 rpy=0 0 0, axis 1 0 0, limit lower=-3.14159 upper=3.14159 effort=0.0 velocity=0.0
- added joint LeftThigh_LeftCalf: type revolute, parent LeftThigh, child LeftCalf, origin xyz=0.2 -0.05 -0.6 rpy=0 0 0, axis 1 0 0, limit lower=-3.14159 upper=3.14159 effort=0.0 velocity=0.0
- added joint RightCalf_RightFoot: type revolute, parent RightCalf, child RightFoot, origin xyz=0 0 -0.5 rpy=0 0 0, axis 1 0 0, limit lower=-3.14159 upper=3.14159 effort=0.0 velocity=0.0
- added joint RightThigh_RightCalf: type revolute, parent RightThigh, child RightCalf, origin xyz=-0.2 -0.05 -0.6 rpy=0 0 0, axis 1 0 0, limit lower=-3.14159 upper=3.14159 effort=0.0 velocity=0.0
- added joint Torso_LeftThigh: type revolute, parent Torso, child LeftThigh, origin xyz=0.4 0 1.85 rpy=0 0 0, axis 1 0 0, limit lower=-3.14159 upper=3.14159 effort=0.0 velocity=0.0
- added joint Torso_RightThigh: type revolute, parent Torso, child RightThigh, origin xyz=-0.4 0 1.85 rpy=0 0 0, axis 1 0 0, limit lower=-3.14159 upper=3.14159 effort=0.0 velocity=0.0

Commit message: Assignment 6

File: body.urdf (robot description, URDF)
Before this commit: robot robot, 9 links, 8 joints
Links:
- removed link BackLeg
- removed link BackLowerLeg
- removed link FrontLeg
- removed link FrontLowerLeg
- removed link LeftLeg
- removed link LeftLowerLeg
- removed link RightLeg
- removed link RightLowerLeg
- removed link Torso
- added link 0, mass 1; collision box size=0.5367997426281297 0.5851819746099385 0.9608173432473253; visual box size=0.5367997426281297 0.5851819746099385 0.9608173432473253
- added link 1, mass 1; collision box size=0.07161382223976787 0.00585468318834137 0.48011826698016646; visual box size=0.07161382223976787 0.00585468318834137 0.48011826698016646
- added link 2, mass 1; collision box size=0.3743431119151851 0.8505187928600575 0.5187108761667947; visual box size=0.3743431119151851 0.8505187928600575 0.5187108761667947
- added link 3, mass 1; collision box size=0.09024777169463682 0.6767363230819874 0.4482552008424595; visual box size=0.09024777169463682 0.6767363230819874 0.4482552008424595
- added link 4, mass 1; collision box size=0.9823400193870006 0.4375947637662092 0.01689721278776668; visual box size=0.9823400193870006 0.4375947637662092 0.01689721278776668
- added link 5, mass 1; collision box size=0.05260938053376374 0.3835415030019975 0.47266569709337247; visual box size=0.05260938053376374 0.3835415030019975 0.47266569709337247
- added link 6, mass 1; collision box size=0.9156242131073808 0.036722784966805144 0.9961234125682681; visual box size=0.9156242131073808 0.036722784966805144 0.9961234125682681
- added link 7, mass 1; collision box size=0.34524082641422105 0.703119808382608 0.3898978674347502; visual box size=0.34524082641422105 0.703119808382608 0.3898978674347502
- added link 8, mass 1; collision box size=0.21293844680583884 0.28001571046472873 0.8462888452988548; visual box size=0.21293844680583884 0.28001571046472873 0.8462888452988548
Joints:
- removed joint BackLeg_BackLowerLeg
- removed joint FrontLeg_FrontLowerLeg
- removed joint LeftLeg_LeftLowerLeg
- removed joint RightLeg_RightLowerLeg
- removed joint Torso_BackLeg
- removed joint Torso_FrontLeg
- removed joint Torso_LeftLeg
- removed joint Torso_RightLeg
- added joint 0_1: type revolute, parent 0, child 1, origin xyz=0.26839987131406484 0 1.4804086716236626 rpy=0 0 0, axis 0 1 0, limit lower=-3.14159 upper=3.14159 effort=0.0 velocity=0.0
- added joint 1_2: type revolute, parent 1, child 2, origin xyz=0.07161382223976787 0 0 rpy=0 0 0, axis 0 1 0, limit lower=-3.14159 upper=3.14159 effort=0.0 velocity=0.0
- added joint 2_3: type revolute, parent 2, child 3, origin xyz=0.3743431119151851 0 0 rpy=0 0 0, axis 0 1 0, limit lower=-3.14159 upper=3.14159 effort=0.0 velocity=0.0
- added joint 3_4: type revolute, parent 3, child 4, origin xyz=0.09024777169463682 0 0 rpy=0 0 0, axis 0 1 0, limit lower=-3.14159 upper=3.14159 effort=0.0 velocity=0.0
- added joint 4_5: type revolute, parent 4, child 5, origin xyz=0.9823400193870006 0 0 rpy=0 0 0, axis 0 1 0, limit lower=-3.14159 upper=3.14159 effort=0.0 velocity=0.0
- added joint 5_6: type revolute, parent 5, child 6, origin xyz=0.05260938053376374 0 0 rpy=0 0 0, axis 0 1 0, limit lower=-3.14159 upper=3.14159 effort=0.0 velocity=0.0
- added joint 6_7: type revolute, parent 6, child 7, origin xyz=0.9156242131073808 0 0 rpy=0 0 0, axis 0 1 0, limit lower=-3.14159 upper=3.14159 effort=0.0 velocity=0.0
- added joint 7_8: type revolute, parent 7, child 8, origin xyz=0.34524082641422105 0 0 rpy=0 0 0, axis 0 1 0, limit lower=-3.14159 upper=3.14159 effort=0.0 velocity=0.0

Commit message: Final done

File: body.urdf (robot description, URDF)
Before this commit: robot robot, 9 links, 8 joints
Links:
- removed link 5
- removed link 6
- removed link 7
- removed link 8
- link 0: geometry collision box size=0.8477835128310957 0.8990085930127647 0.4689208230331047; visual box size=0.8477835128310957 0.8990085930127647 0.4689208230331047
- link 1: geometry collision box size=0.199066172139015 0.5059150223500399 0.6670897978966985; visual box size=0.199066172139015 0.5059150223500399 0.6670897978966985
- link 2: geometry collision box size=0.977717262523462 0.12348470965742286 0.8436371922446059; visual box size=0.977717262523462 0.12348470965742286 0.8436371922446059
- link 3: geometry collision box size=0.5086944872784408 0.949440928052879 0.349997569265346; visual box size=0.5086944872784408 0.949440928052879 0.349997569265346
- link 4: geometry collision box size=0.6271523938064931 0.7002218427065944 0.6171277694448312; visual box size=0.6271523938064931 0.7002218427065944 0.6171277694448312
Joints:
- removed joint 4_5
- removed joint 5_6
- removed joint 6_7
- removed joint 7_8
- joint 0_1: origin xyz=0.26839987131406484 0 1.4804086716236626 rpy=0 0 0 -> xyz=0.4238917564155478 0 1.2344604115165523 rpy=0 0 0
- joint 1_2: origin xyz=0.07161382223976787 0 0 rpy=0 0 0 -> xyz=0.199066172139015 0 0 rpy=0 0 0
- joint 2_3: origin xyz=0.3743431119151851 0 0 rpy=0 0 0 -> xyz=0.977717262523462 0 0 rpy=0 0 0
- joint 3_4: origin xyz=0.09024777169463682 0 0 rpy=0 0 0 -> xyz=0.5086944872784408 0 0 rpy=0 0 0

Commit message: SPAWNS CORRECTLY

File: body.urdf (robot description, URDF)
Before this commit: robot robot, 5 links, 4 joints
Links:
- added link 10, mass 1; collision box size=0.2546784140696443 0.9501328591142532 0.017288994516915006; visual box size=0.2546784140696443 0.9501328591142532 0.017288994516915006
- added link 11, mass 1; collision box size=0.049386667048118886 0.07905161395075909 0.03371537384552802; visual box size=0.049386667048118886 0.07905161395075909 0.03371537384552802
- added link 5, mass 1; collision box size=0.888878716050141 0.3437440407376028 0.6475818653148381; visual box size=0.888878716050141 0.3437440407376028 0.6475818653148381
- added link 6, mass 1; collision box size=0.29130185038102974 0.41317013521804646 0.01657683211334015; visual box size=0.29130185038102974 0.41317013521804646 0.01657683211334015
- added link 7, mass 1; collision box size=0.40294576109563063 0.6987596476445344 0.33641828822301756; visual box size=0.40294576109563063 0.6987596476445344 0.33641828822301756
- added link 8, mass 1; collision box size=0.23037018801558717 0.22735821540137513 0.34240801390270703; visual box size=0.23037018801558717 0.22735821540137513 0.34240801390270703
- added link 9, mass 1; collision box size=0.7801236259773219 0.08257135183057406 0.9543705229219199; visual box size=0.7801236259773219 0.08257135183057406 0.9543705229219199
- link 0: geometry collision box size=0.2618348923677382 0.22502097114233593 1.128157025780047; visual box size=0.2618348923677382 0.22502097114233593 1.128157025780047
- link 1: geometry collision box size=0.7388568957299277 0.2693414055838303 1.0677094631750623; visual box size=0.7388568957299277 0.2693414055838303 1.0677094631750623
- link 2: geometry collision box size=0.5884293886128591 0.1917617973950143 0.3266059085798054; visual box size=0.5884293886128591 0.1917617973950143 0.3266059085798054
- link 3: geometry collision box size=0.019468828957058475 0.22555764225752173 0.6975802316583536; visual box size=0.019468828957058475 0.22555764225752173 0.6975802316583536
- link 4: geometry collision box size=0.28632038551844496 0.46862307594824415 0.5994881933746432; visual box size=0.28632038551844496 0.46862307594824415 0.5994881933746432
Joints:
- removed joint 2_3
- removed joint 3_4
- added joint 1_3: type revolute, parent 1, child 3, origin xyz=0.0 -0.2693414055838303 0.0 rpy=0 0 0, axis 0 1 0, limit lower=-3.14159 upper=3.14159 effort=0.0 velocity=0.0
- added joint 1_9: type revolute, parent 1, child 9, origin xyz=-0.36942844786496387 -0.13467070279191515 0.0 rpy=0 0 0, axis 0 1 0, limit lower=-3.14159 upper=3.14159 effort=0.0 velocity=0.0
- added joint 2_4: type revolute, parent 2, child 4, origin xyz=0.5884293886128591 0.0 0.0 rpy=0 0 0, axis 0 1 0, limit lower=-3.14159 upper=3.14159 effort=0.0 velocity=0.0
- added joint 3_5: type revolute, parent 3, child 5, origin xyz=0.0 -0.22555764225752173 0.0 rpy=0 0 0, axis 0 1 0, limit lower=-3.14159 upper=3.14159 effort=0.0 velocity=0.0
- added joint 4_11: type revolute, parent 4, child 11, origin xyz=0.14316019275922248 0.23431153797412207 0.0 rpy=0 0 0, axis 0 1 0, limit lower=-3.14159 upper=3.14159 effort=0.0 velocity=0.0
- added joint 4_7: type revolute, parent 4, child 7, origin xyz=0.14316019275922248 -0.23431153797412207 0.0 rpy=0 0 0, axis 0 1 0, limit lower=-3.14159 upper=3.14159 effort=0.0 velocity=0.0
- added joint 5_10: type revolute, parent 5, child 10, origin xyz=0.0 -0.3437440407376028 0.0 rpy=0 0 0, axis 0 1 0, limit lower=-3.14159 upper=3.14159 effort=0.0 velocity=0.0
- added joint 5_6: type revolute, parent 5, child 6, origin xyz=-0.4444393580250705 -0.1718720203688014 0.0 rpy=0 0 0, axis 0 1 0, limit lower=-3.14159 upper=3.14159 effort=0.0 velocity=0.0
- added joint 5_8: type revolute, parent 5, child 8, origin xyz=0.4444393580250705 -0.1718720203688014 0.0 rpy=0 0 0, axis 0 1 0, limit lower=-3.14159 upper=3.14159 effort=0.0 velocity=0.0
- joint 0_1: origin xyz=0.4238917564155478 0 1.2344604115165523 rpy=0 0 0 -> xyz=0.0 -0.11251048557116797 1.5640785128900236 rpy=0 0 0
- joint 1_2: origin xyz=0.199066172139015 0 0 rpy=0 0 0 -> xyz=0.36942844786496387 -0.13467070279191515 0.0 rpy=0 0 0
